File: Cobble-board-test/Cobble-board-test.kicad_pcb (KiCad board)
At the start: 2 copper layers, 46 x 45 mm, 16 parts, among them J2 JST PH2.0 Battery, J3 Stemma PH, J4 Grove, Q1 SI2302DS, SW1 SW_Push, SW3 SW_VIBE, SW4 MSK22D27

Commit message: Cobbl-board-test is complete and tested
Parts:
- SW4: value MSK22D27 -> DPDT
Routing:
- net 3V3: track 78.9 -> 81.5 mm
- net Net-(U1-ChrgBst-Pad41): track 0.00 -> 1.30 mm
Other:
- board text added: "Vibe sensor pad is too small SW1 pin spacing is wrong Light sensor is wired to a pin that does not support ADC"
